File: vga-sync-separator2-3.3V.brd (EAGLE design)
At the start: 66 x 44 mm, 14 parts, among them U1 EL1883, U2 AMS1117-3.3, X1 VGA-PORT, X2 VGA-PORT

Commit message: Add files via upload
Parts:
- moved C4 30.6 mm to (20.0, 40.0), turned to 180 degrees
- moved R2 26.9 mm to (19.0, 35.0), turned to 90 degrees
- moved R3 23.8 mm to (22.0, 35.0), turned to 90 degrees
- moved C3 20.9 mm to (25.0, 35.0), turned to 270 degrees
Routing:
- net CSYNC-IN: track 34.0 -> 20.9 mm
- net N$1: track 18.7 -> 7.86 mm
- net B: track 46.8 -> 55.4 mm, vias 1 -> 0
- net 5V: track 25.3 -> 22.2 mm, vias 1 -> 0
- net G: track 49.3 -> 47.3 mm, vias 1 -> 0
- net N$2: track 9.60 -> 10.5 mm
- net R: track 51.7 -> 52.5 mm, vias 1 -> 0
- net HSYNC-OUT: track 44.4 -> 44.5 mm, vias 1 -> 0
- added copper zone on layer 1, net 5V
